Commit message: Custom USD drifts with the ocean current
Signed-off-by: Alejandro Hernandez Cordero <ahcorde@gmail.com>

File: kai_custom_vehicle/models/custom_usv/model.sdf.xacro (robot description, xacro)
@@ -42,7 +42,11 @@
        are what the boat bumps with. The same box is marked gz:wind="true":
        the wind system pushes on the part of it above the waterline, so a
-       wind in the world sets the boat drifting and turning. -->
+       wind in the world sets the boat drifting and turning. And it is
+       marked gz:ocean_current="true": the ocean current system drags the
+       part below the waterline against the water, so the boat drifts with
+       the world's current. -->
   <xacro:macro name="pontoon" params="side y">
-    <collision name="pontoon_${side}" gz:buoyancy="true" gz:wind="true">
+    <collision name="pontoon_${side}" gz:buoyancy="true" gz:wind="true"
+               gz:ocean_current="true">
       <pose>0 ${y} ${hull_z} 0 0 0</pose>
       <geometry>
@@ -130,17 +134,18 @@
     <xacro:thruster side="stbd" coefficient="-0.02"/>
     <!-- ===================== Hydrodynamics =====================
-         Fossen damping on base_link. Placeholder surface-vessel coefficients,
-         the magnitudes the BlueBoat uses: strong sway and yaw resistance,
-         moderate surge, and heave, roll and pitch damping so the boat settles
-         on the buoyancy instead of bobbing. Tune them against the real
-         vehicle. -->
+         Fossen damping on base_link, for the motions the water's drag on the
+         marked pontoons does not cover: heave, roll, pitch and yaw, so the
+         boat settles on the buoyancy instead of bobbing and does not spin
+         freely. Surge and sway are left out on purpose: the pontoons'
+         gz:ocean_current marks provide them, against the water, and Fossen
+         terms on the same axes would damp the boat against the ground as
+         well and hold it back in a current. Placeholder coefficients, the
+         magnitudes the BlueBoat uses; tune them against the real vehicle. -->
     <plugin filename="gz-sim-hydrodynamics-system"
             name="gz::sim::systems::Hydrodynamics">
       <link_name>base_link</link_name>
       <water_density>${water_density}</water_density>
-      <xU>-20</xU>    <yV>-40</yV>    <zW>-30</zW>
+      <zW>-30</zW>
       <kP>-20</kP>    <mQ>-20</mQ>    <nR>-15</nR>
-      <xUabsU>-30</xUabsU>
-      <yVabsV>-90</yVabsV>
       <zWabsW>-100</zWabsW>
       <kPabsP>-40</kPabsP>

Commit message: demo
Signed-off-by: Alejandro Hernandez Cordero <ahcorde@gmail.com>

File: kai_custom_vehicle/models/custom_usv/model.sdf.xacro (robot description, xacro)
@@ -134,7 +134,8 @@
          moderate surge, and heave, roll and pitch damping so the boat settles
          on the buoyancy instead of bobbing. Tune them against the real
-         vehicle. -->
-    <plugin filename="gz-sim-hydrodynamics-system"
-            name="gz::sim::systems::Hydrodynamics">
+         vehicle. gz_hydrodynamics damps against the water rather than the
+         ground, so the boat drifts with the world's ocean current. -->
+    <plugin filename="gz-maritime-hydrodynamics-system"
+            name="gz::sim::maritime::Hydrodynamics">
       <link_name>base_link</link_name>
       <water_density>${water_density}</water_density>
@@ -148,22 +149,10 @@
       <nRabsR>-30</nRabsR>
     </plugin>
-    <!-- Added mass: water accelerated along with the hull. Gazebo takes it as
-         <fluid_added_mass> inside a link's <inertial> (SDF 1.11 and later),
-         which cannot live in the URDF: URDF has no such element, and a merged
-         include cannot amend base_link's inertial from here. Left out, since
-         it is small for a boat this size at these speeds. In a link written
-         in SDF it would read, with values to be identified for the hull:
-         <inertial>
-           <mass>12</mass>
-           <fluid_added_mass>
-             <xx>0.6</xx>
-             <yy>6.0</yy>
-             <zz>12.0</zz>
-             <pp>0.1</pp>
-             <qq>0.5</qq>
-             <rr>0.5</rr>
-           </fluid_added_mass>
-         </inertial>
-    -->
+    <!-- Added mass: water accelerated along with the hull. It goes in the
+         plugin above as <xDotU>, <yDotV>, <zDotW>, <kDotP>, <mDotQ> and
+         <nDotR>, not as SDF <fluid_added_mass>, which only DART implements.
+         Left out, since it is small for a boat this size at these speeds,
+         and plugin added mass turns a step in the current into a force
+         spike. -->
     <!-- ===================== Sensors =====================
          They need the world to run the sensors, IMU, magnetometer and NavSat
